Commit message: Update biped.urdf.xacro to adjust joint limits and add ROS2 control configuration

File: rsa_biped/urdf/biped.urdf.xacro (robot description, xacro)
@@ -86,5 +86,5 @@
         <child link="left_ankle_link_servo_motor_link" />
         <axis xyz="0 0 1" />
-        <limit lower="-${PI/2}" upper="${PI/2}" effort="1000" velocity="0.1" />
+        <limit lower="-${PI}" upper="${PI}" effort="1000" velocity="0.1" />
     </joint>
     <!-- Left Ankle -->
@@ -153,7 +153,41 @@
         <child link="right_ankle_link_servo_motor_link" />
         <axis xyz="0 0 1" />
-        <limit lower="-${PI/2}" upper="${PI/2}" effort="1000" velocity="0.1" />
+        <limit lower="-${PI}" upper="${PI}" effort="1000" velocity="0.1" />
     </joint>
     <!-- Right Ankle -->
     <xacro:right_ankle parent_link="right_foot_servo_link" xyz="-0.01 -0.01 -0.0225" rpy="${PI} 0 -${PI/2}" />
+    <!-- ========================================================== -->
+    <!-- ========================================================== -->
+    <!-- ===============        ROS2 Control        =============== -->
+    <!-- ========================================================== -->
+    <!-- ========================================================== -->
+    <ros2_control name="biped_ros2_control" type="system">
+        <hardware>
+            <plugin>fake_components/GenericSystem</plugin>
+        </hardware>
+        <joint name="left_hip_knee_joint_1">
+            <command_interface name="position" />
+            <state_interface name="position" />
+        </joint>
+        <joint name="left_hip_knee_joint_2">
+            <command_interface name="position" />
+            <state_interface name="position" />
+        </joint>
+        <joint name="left_ankle_joint">
+            <command_interface name="position" />
+            <state_interface name="position" />
+        </joint>
+        <joint name="right_hip_knee_joint_1">
+            <command_interface name="position" />
+            <state_interface name="position" />
+        </joint>
+        <joint name="right_hip_knee_joint_2">
+            <command_interface name="position" />
+            <state_interface name="position" />
+        </joint>
+        <joint name="right_ankle_joint">
+            <command_interface name="position" />
+            <state_interface name="position" />
+        </joint>
+    </ros2_control>
 </robot>
